File: adapter/adapter.sch (KiCad schematic (older format))
At the start: 2 parts, among them J1 eurocard_ab_female, J2 Conn_02x25_Odd_Even

Commit message: Update to adapter.
Connections:
- wire segments 72 -> 76
Changed lines of the file:
@@
 Text Label 3950 4700 0    50   ~ 0
 ~RD~
+$Comp
+L power:GND #PWR?
+U 1 1 5F9D596B
+P 3300 3000
+F 0 "#PWR?" H 3300 2750 50  0001 C CNN
+F 1 "GND" V 3305 2872 50  0000 R CNN
+F 2 "" H 3300 3000 50  0001 C CNN
+F 3 "" H 3300 3000 50  0001 C CNN
+	1    3300 3000
+	0    1    1    0
+$EndComp
+Wire Wire Line
+	3450 3000 3300 3000
+$Comp
+L power:GND #PWR?
+U 1 1 5F9D85CA
+P 4050 2150
+F 0 "#PWR?" H 4050 1900 50  0001 C CNN
+F 1 "GND" V 4055 2022 50  0000 R CNN
+F 2 "" H 4050 2150 50  0001 C CNN
+F 3 "" H 4050 2150 50  0001 C CNN
+	1    4050 2150
+	0    -1   -1   0
+$EndComp
+Wire Wire Line
+	3850 2200 3900 2200
+Wire Wire Line
+	3900 2200 3950 2150
+Wire Wire Line
+	3950 2150 4050 2150
 $EndSCHEMATC
