File: eagle_files/james_z80_debug_mod.brd (EAGLE design)
At the start: 160 x 100 mm, 50 parts, among them IC1 74LS32N, IC10 74HC573N, IC11 27C128P, IC13 74LS245N, IC14 74LS245N, IC15 74LS245N, IC16 74HC125N, IC2 74LS04N, IC3 74LS139N, IC4 74HC573N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

Commit message: Update monitor mods.
Connections:
- net GND: now also IC9.14
Changed lines of the file:
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@@
 <contactref element="IC10" pad="8"/>
 <contactref element="IC10" pad="9"/>
+<contactref element="IC9" pad="14"/>
 <wire x1="-261.62" y1="25.4" x2="-261.62" y2="15.24" width="0" layer="19" extent="1-1"/>
 <wire x1="-266.7" y1="25.4" x2="-261.62" y2="25.4" width="0" layer="19" extent="1-1"/>
@@
 <wire x1="-66.04" y1="12.7" x2="-66.04" y2="-15.24" width="0" layer="19" extent="1-1"/>
 <wire x1="-73.66" y1="38.1" x2="-66.04" y2="12.7" width="0" layer="19" extent="1-1"/>
-<wire x1="-25.4" y1="38.1" x2="-33.02" y2="2.54" width="0" layer="19" extent="1-1"/>
+<wire x1="-25.4" y1="35.56" x2="-33.02" y2="2.54" width="0" layer="19" extent="1-1"/>
+<wire x1="-25.4" y1="38.1" x2="-25.4" y2="35.56" width="0" layer="19" extent="1-1"/>
 <wire x1="-142.24" y1="40.64" x2="-119.38" y2="2.54" width="0" layer="19" extent="1-1"/>
 <wire x1="-2.54" y1="-130.81" x2="-15.24" y2="-43.18" width="0" layer="19" extent="1-1"/>

Commit message: Add a label to eagle schematics.
Connections:
- net N$4 renamed !Y_IORQ
Changed lines of the file:
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@@
 <wire x1="-99.06" y1="-22.86" x2="-149.86" y2="3.81" width="0" layer="19" extent="1-1"/>
 </signal>
-<signal name="N$4">
+<signal name="!Y_IORQ">
 <contactref element="IC10" pad="16"/>
 <contactref element="IC7" pad="5"/>
