File: monitor/z80_monitor/z80_monitor.kicad_pcb (KiCad board)
At the start: 2 copper layers, 15 parts, among them J1 Conn_02x25_Odd_Even, U1 74HC237, U10 74HCT365, U11 74HC573, U12 74LS05, U2 74HCT245, U3 74HC573, U4 74LS04, U5 74HC32, U6 74LS00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

Commit message: More updates.
Parts:
- added U13: ATmega328P-PU, Housings_DIP:DIP-28_W7.62mm, F.Cu at (118.1, 48.3)
- moved U5 37.7 mm to (132.1, 61.0)
- moved U12 28.5 mm to (160.0, 63.5)
- moved U9 19.1 mm to (160.0, 85.1)
- moved U11 3.81 mm to (160.0, 34.3)
Changed lines of the file:
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@@
     (tracks 0)
     (zones 0)
-    (modules 15)
-    (nets 93)
+    (modules 16)
+    (nets 120)
   )
   (page A4)
@@
   (net 91 "Net-(U11-Pad19)")
   (net 92 "Net-(U12-Pad8)")
+  (net 93 "Net-(U13-Pad1)")
+  (net 94 "Net-(U13-Pad15)")
+  (net 95 "Net-(U13-Pad2)")
+  (net 96 "Net-(U13-Pad16)")
+  (net 97 "Net-(U13-Pad3)")
+  (net 98 "Net-(U13-Pad17)")
+  (net 99 "Net-(U13-Pad4)")
+  (net 100 "Net-(U13-Pad18)")
+  (net 101 "Net-(U13-Pad5)")
+  (net 102 "Net-(U13-Pad19)")
+  (net 103 "Net-(U13-Pad6)")
+  (net 104 "Net-(U13-Pad20)")
+  (net 105 "Net-(U13-Pad7)")
+  (net 106 "Net-(U13-Pad21)")
+  (net 107 "Net-(U13-Pad22)")
+  (net 108 "Net-(U13-Pad9)")
+  (net 109 "Net-(U13-Pad23)")
+  (net 110 "Net-(U13-Pad10)")
+  (net 111 "Net-(U13-Pad24)")
+  (net 112 "Net-(U13-Pad11)")
+  (net 113 "Net-(U13-Pad25)")
+  (net 114 "Net-(U13-Pad12)")
+  (net 115 "Net-(U13-Pad26)")
+  (net 116 "Net-(U13-Pad13)")
+  (net 117 "Net-(U13-Pad27)")
+  (net 118 "Net-(U13-Pad14)")
+  (net 119 "Net-(U13-Pad28)")
   (net_class Default "This is the default net class."
     (clearance 0.2)
@@
     (add_net "Net-(U11-Pad19)")
     (add_net "Net-(U12-Pad8)")
+    (add_net "Net-(U13-Pad1)")
+    (add_net "Net-(U13-Pad10)")
+    (add_net "Net-(U13-Pad11)")
+    (add_net "Net-(U13-Pad12)")
+    (add_net "Net-(U13-Pad13)")
+    (add_net "Net-(U13-Pad14)")
+    (add_net "Net-(U13-Pad15)")
+    (add_net "Net-(U13-Pad16)")
+    (add_net "Net-(U13-Pad17)")
+    (add_net "Net-(U13-Pad18)")
+    (add_net "Net-(U13-Pad19)")
+    (add_net "Net-(U13-Pad2)")
+    (add_net "Net-(U13-Pad20)")
+    (add_net "Net-(U13-Pad21)")
+    (add_net "Net-(U13-Pad22)")
+    (add_net "Net-(U13-Pad23)")
+    (add_net "Net-(U13-Pad24)")
+    (add_net "Net-(U13-Pad25)")
+    (add_net "Net-(U13-Pad26)")
+    (add_net "Net-(U13-Pad27)")
+    (add_net "Net-(U13-Pad28)")
+    (add_net "Net-(U13-Pad3)")
+    (add_net "Net-(U13-Pad4)")
+    (add_net "Net-(U13-Pad5)")
+    (add_net "Net-(U13-Pad6)")
+    (add_net "Net-(U13-Pad7)")
+    (add_net "Net-(U13-Pad9)")
     (add_net "Net-(U2-Pad19)")
     (add_net "Net-(U3-Pad1)")
@@
     (add_net "Net-(U9-Pad14)")
   )
+  (module Housings_DIP:DIP-28_W7.62mm (layer F.Cu)
+    (at 118.11 48.26)
+    (descr "28-lead though-hole mounted DIP package, row spacing 7.62 mm (300 mils)")
+    (tags "THT DIP DIL PDIP 2.54mm 7.62mm 300mil")
+    (fp_text reference U13 (at 3.81 -2.33) (layer F.SilkS)
+      (effects (font (size 1 1) (thickness 0.15)))
+    )
+    (fp_text value ATmega328P-PU (at 3.81 35.35) (layer F.Fab)
+      (effects (font (size 1 1) (thickness 0.15)))
+    )
+    (fp_line (start 8.7 -1.55) (end -1.1 -1.55) (layer F.CrtYd) (width 0.05))
+    (fp_line (start 8.7 34.55) (end 8.7 -1.55) (layer F.CrtYd) (width 0.05))
+    (fp_line (start -1.1 34.55) (end 8.7 34.55) (layer F.CrtYd) (width 0.05))
+    (fp_line (start -1.1 -1.55) (end -1.1 34.55) (layer F.CrtYd) (width 0.05))
+    (fp_line (start 6.46 -1.33) (end 4.81 -1.33) (layer F.SilkS) (width 0.12))
+    (fp_line (start 6.46 34.35) (end 6.46 -1.33) (layer F.SilkS) (width 0.12))
+    (fp_line (start 1.16 34.35) (end 6.46 34.35) (layer F.SilkS) (width 0.12))
+    (fp_line (start 1.16 -1.33) (end 1.16 34.35) (layer F.SilkS) (width 0.12))
+    (fp_line (start 2.81 -1.33) (end 1.16 -1.33) (layer F.SilkS) (width 0.12))
+    (fp_line (start 0.635 -0.27) (end 1.635 -1.27) (layer F.Fab) (width 0.1))
+    (fp_line (start 0.635 34.29) (end 0.635 -0.27) (layer F.Fab) (width 0.1))
+    (fp_line (start 6.985 34.29) (end 0.635 34.29) (layer F.Fab) (width 0.1))
+    (fp_line (start 6.985 -1.27) (end 6.985 34.29) (layer F.Fab) (width 0.1))
+    (fp_line (start 1.635 -1.27) (end 6.985 -1.27) (layer F.Fab) (width 0.1))
+    (fp_arc (start 3.81 -1.33) (end 2.81 -1.33) (angle -180) (layer F.SilkS) (width 0.12))
+    (fp_text user %R (at 3.81 16.51) (layer F.Fab)
+      (effects (font (size 1 1) (thickness 0.15)))
+    )
+    (pad 1 thru_hole rect (at 0 0) (size 1.6 1.6) (drill 0.8) (layers *.Cu *.Mask)
+      (net 93 "Net-(U13-Pad1)"))
+    (pad 15 thru_hole oval (at 7.62 33.02) (size 1.6 1.6) (drill 0.8) (layers *.Cu *.Mask)
+      (net 94 "Net-(U13-Pad15)"))
+    (pad 2 thru_hole oval (at 0 2.54) (size 1.6 1.6) (drill 0.8) (layers *.Cu *.Mask)
+      (net 95 "Net-(U13-Pad2)"))
+    (pad 16 thru_hole oval (at 7.62 30.48) (size 1.6 1.6) (drill 0.8) (layers *.Cu *.Mask)
+      (net 96 "Net-(U13-Pad16)"))
+    (pad 3 thru_hole oval (at 0 5.08) (size 1.6 1.6) (drill 0.8) (layers *.Cu *.Mask)
+      (net 97 "Net-(U13-Pad3)"))
+    (pad 17 thru_hole oval (at 7.62 27.94) (size 1.6 1.6) (drill 0.8) (layers *.Cu *.Mask)
+      (net 98 "Net-(U13-Pad17)"))
+    (pad 4 thru_hole oval (at 0 7.62) (size 1.6 1.6) (drill 0.8) (layers *.Cu *.Mask)
+      (net 99 "Net-(U13-Pad4)"))
+    (pad 18 thru_hole oval (at 7.62 25.4) (size 1.6 1.6) (drill 0.8) (layers *.Cu *.Mask)
+      (net 100 "Net-(U13-Pad18)"))
+    (pad 5 thru_hole oval (at 0 10.16) (size 1.6 1.6) (drill 0.8) (layers *.Cu *.Mask)
+      (net 101 "Net-(U13-Pad5)"))
+    (pad 19 thru_hole oval (at 7.62 22.86) (size 1.6 1.6) (drill 0.8) (layers *.Cu *.Mask)
+      (net 102 "Net-(U13-Pad19)"))
+    (pad 6 thru_hole oval (at 0 12.7) (size 1.6 1.6) (drill 0.8) (layers *.Cu *.Mask)
+      (net 103 "Net-(U13-Pad6)"))
+    (pad 20 thru_hole oval (at 7.62 20.32) (size 1.6 1.6) (drill 0.8) (layers *.Cu *.Mask)
+      (net 104 "Net-(U13-Pad20)"))
+    (pad 7 thru_hole oval (at 0 15.24) (size 1.6 1.6) (drill 0.8) (layers *.Cu *.Mask)
+      (net 105 "Net-(U13-Pad7)"))
+    (pad 21 thru_hole oval (at 7.62 17.78) (size 1.6 1.6) (drill 0.8) (layers *.Cu *.Mask)
+      (net 106 "Net-(U13-Pad21)"))
+    (pad 8 thru_hole oval (at 0 17.78) (size 1.6 1.6) (drill 0.8) (layers *.Cu *.Mask)
+      (net 107 "Net-(U13-Pad22)"))
+    (pad 22 thru_hole oval (at 7.62 15.24) (size 1.6 1.6) (drill 0.8) (layers *.Cu *.Mask)
+      (net 107 "Net-(U13-Pad22)"))
+    (pad 9 thru_hole oval (at 0 20.32) (size 1.6 1.6) (drill 0.8) (layers *.Cu *.Mask)
+      (net 108 "Net-(U13-Pad9)"))
+    (pad 23 thru_hole oval (at 7.62 12.7) (size 1.6 1.6) (drill 0.8) (layers *.Cu *.Mask)
+      (net 109 "Net-(U13-Pad23)"))
+    (pad 10 thru_hole oval (at 0 22.86) (size 1.6 1.6) (drill 0.8) (layers *.Cu *.Mask)
+      (net 110 "Net-(U13-Pad10)"))
+    (pad 24 thru_hole oval (at 7.62 10.16) (size 1.6 1.6) (drill 0.8) (layers *.Cu *.Mask)
+      (net 111 "Net-(U13-Pad24)"))
+    (pad 11 thru_hole oval (at 0 25.4) (size 1.6 1.6) (drill 0.8) (layers *.Cu *.Mask)
+      (net 112 "Net-(U13-Pad11)"))
+    (pad 25 thru_hole oval (at 7.62 7.62) (size 1.6 1.6) (drill 0.8) (layers *.Cu *.Mask)
+      (net 113 "Net-(U13-Pad25)"))
+    (pad 12 thru_hole oval (at 0 27.94) (size 1.6 1.6) (drill 0.8) (layers *.Cu *.Mask)
+      (net 114 "Net-(U13-Pad12)"))
+    (pad 26 thru_hole oval (at 7.62 5.08) (size 1.6 1.6) (drill 0.8) (layers *.Cu *.Mask)
+      (net 115 "Net-(U13-Pad26)"))
+    (pad 13 thru_hole oval (at 0 30.48) (size 1.6 1.6) (drill 0.8) (layers *.Cu *.Mask)
+      (net 116 "Net-(U13-Pad13)"))
+    (pad 27 thru_hole oval (at 7.62 2.54) (size 1.6 1.6) (drill 0.8) (layers *.Cu *.Mask)
+      (net 117 "Net-(U13-Pad27)"))
+    (pad 14 thru_hole oval (at 0 33.02) (size 1.6 1.6) (drill 0.8) (layers *.Cu *.Mask)
+      (net 118 "Net-(U13-Pad14)"))
+    (pad 28 thru_hole oval (at 7.62 0) (size 1.6 1.6) (drill 0.8) (layers *.Cu *.Mask)
+      (net 119 "Net-(U13-Pad28)"))
+    (model ${KISYS3DMOD}/Housings_DIP.3dshapes/DIP-28_W7.62mm.wrl
+      (at (xyz 0 0 0))
+      (scale (xyz 1 1 1))
+      (rotate (xyz 0 0 0))
+    )
+  )
   (module Housings_DIP:DIP-14_W7.62mm (layer F.Cu)
-    (at 144.78 87.63)
+    (at 160.02 63.5)
     (descr "14-lead though-hole mounted DIP package, row spacing 7.62 mm (300 mils)")
     (tags "THT DIP DIL PDIP 2.54mm 7.62mm 300mil")
@@
   )
   (module Housings_DIP:DIP-20_W7.62mm (layer F.Cu)
-    (at 160.02 38.1)
+    (at 160.02 34.29)
     (descr "20-lead though-hole mounted DIP package, row spacing 7.62 mm (300 mils)")
     (tags "THT DIP DIL PDIP 2.54mm 7.62mm 300mil")
@@
   )
   (module Housings_DIP:DIP-16_W7.62mm (layer F.Cu)
-    (at 158.75 66.04)
+    (at 160.02 85.09)
     (descr "16-lead though-hole mounted DIP package, row spacing 7.62 mm (300 mils)")
     (tags "THT DIP DIL PDIP 2.54mm 7.62mm 300mil")
@@
   )
   (module Housings_DIP:DIP-14_W7.62mm (layer F.Cu)
-    (at 158.75 87.63)
+    (at 132.08 60.96)
     (descr "14-lead though-hole mounted DIP package, row spacing 7.62 mm (300 mils)")
     (tags "THT DIP DIL PDIP 2.54mm 7.62mm 300mil")
