File: kicad/z80_monitor.sch (KiCad schematic (older format))
At the start: 30 parts, among them J1 Conn_01x06, J2 Conn_02x03_Odd_Even, J3 Conn_02x25_Odd_Even, U1 ADuM1201CR, U2 ATmega1281-16AU, Y1 16MHz

Commit message: Update LED resistor values to try to match brightness.
Parts:
- R1, R4: value 1K0 -> 6K2
- R3: value 1K0 -> 2K7
- R5, R6: value 1K0 -> 1K8
- R7: value 1K0 -> 3K3
Changed lines of the file:
@@
 P 2000 5350
 F 0 "R1" H 2059 5396 50  0000 L CNN
-F 1 "1K0" H 2059 5305 50  0000 L CNN
+F 1 "6K2" H 2059 5305 50  0000 L CNN
 F 2 "Resistor_SMD:R_0603_1608Metric_Pad1.05x0.95mm_HandSolder" H 2000 5350 50  0001 C CNN
 F 3 "~" H 2000 5350 50  0001 C CNN
@@
 P 8850 1550
 F 0 "R4" H 8909 1596 50  0000 L CNN
-F 1 "1K0" H 8909 1505 50  0000 L CNN
+F 1 "6K2" H 8909 1505 50  0000 L CNN
 F 2 "Resistor_SMD:R_0603_1608Metric_Pad1.05x0.95mm_HandSolder" H 8850 1550 50  0001 C CNN
 F 3 "~" H 8850 1550 50  0001 C CNN
@@
 P 9200 1550
 F 0 "R5" H 9259 1596 50  0000 L CNN
-F 1 "1K0" H 9259 1505 50  0000 L CNN
+F 1 "1K8" H 9259 1505 50  0000 L CNN
 F 2 "Resistor_SMD:R_0603_1608Metric_Pad1.05x0.95mm_HandSolder" H 9200 1550 50  0001 C CNN
 F 3 "~" H 9200 1550 50  0001 C CNN
@@
 P 9550 1550
 F 0 "R6" H 9609 1596 50  0000 L CNN
-F 1 "1K0" H 9609 1505 50  0000 L CNN
+F 1 "1K8" H 9609 1505 50  0000 L CNN
 F 2 "Resistor_SMD:R_0603_1608Metric_Pad1.05x0.95mm_HandSolder" H 9550 1550 50  0001 C CNN
 F 3 "~" H 9550 1550 50  0001 C CNN
@@
 P 6400 3500
 F 0 "R3" H 6459 3546 50  0000 L CNN
-F 1 "1K0" H 6459 3455 50  0000 L CNN
+F 1 "2K7" H 6459 3455 50  0000 L CNN
 F 2 "Resistor_SMD:R_0603_1608Metric_Pad1.05x0.95mm_HandSolder" H 6400 3500 50  0001 C CNN
 F 3 "~" H 6400 3500 50  0001 C CNN
@@
 P 9900 1550
 F 0 "R7" H 9959 1596 50  0000 L CNN
-F 1 "1K0" H 9959 1505 50  0000 L CNN
+F 1 "3K3" H 9959 1505 50  0000 L CNN
 F 2 "Resistor_SMD:R_0603_1608Metric_Pad1.05x0.95mm_HandSolder" H 9900 1550 50  0001 C CNN
 F 3 "~" H 9900 1550 50  0001 C CNN
