File: kicad/z80_monitor.kicad_pcb (KiCad board)
At the start: 2 copper layers, 42.5 x 74.9 mm, 30 parts, among them J1 Conn_01x06, J2 Conn_02x03_Odd_Even, J3 Conn_02x25_Odd_Even, U1 ADuM1201CR, U2 ATmega1281-16AU, Y1 16MHz

Commit message: Update gerbers.
Other:
- board text added: "1"
Changed lines of the file:
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@@
   (general
     (thickness 1.6)
-    (drawings 14)
+    (drawings 16)
     (tracks 756)
     (zones 0)
@@
     )
   )
+  (gr_text 1 (at 116.84 69.215) (layer F.SilkS)
+    (effects (font (size 1.5 1.5) (thickness 0.3)))
+  )
+  (gr_text 1 (at 104.14 116.205) (layer F.SilkS)
+    (effects (font (size 1.5 1.5) (thickness 0.3)))
+  )
   (gr_arc (start 144.145 125.73) (end 144.145 126.365) (angle -90) (layer Edge.Cuts) (width 0.1))
   (gr_arc (start 102.87 125.73) (end 102.235 125.73) (angle -90) (layer Edge.Cuts) (width 0.1))
@@
     (effects (font (size 1.5 1.5) (thickness 0.3)))
   )
-  (gr_text COMS (at 111.125 53.34) (layer F.Cu)
+  (gr_text COMS (at 111.125 53.34) (layer F.SilkS)
     (effects (font (size 1 1) (thickness 0.25)))
   )
-  (gr_text PWR (at 106.045 53.34) (layer F.Cu)
+  (gr_text PWR (at 106.045 53.34) (layer F.SilkS)
     (effects (font (size 1 1) (thickness 0.25)))
   )
-  (gr_text REQ (at 116.205 53.34) (layer F.Cu)
+  (gr_text REQ (at 116.205 53.34) (layer F.SilkS)
     (effects (font (size 1 1) (thickness 0.25)))
   )
-  (gr_text ACK (at 121.285 53.34) (layer F.Cu)
+  (gr_text ACK (at 121.285 53.34) (layer F.SilkS)
     (effects (font (size 1 1) (thickness 0.25)))
   )
-  (gr_text HALT (at 125.73 53.34) (layer F.Cu)
+  (gr_text HALT (at 125.73 53.34) (layer F.SilkS)
     (effects (font (size 1 1) (thickness 0.25)))
   )

Commit message: Update board
Parts:
- R1, R4: value 1K0 -> 6K2
- R3: value 1K0 -> 2K7
- R5, R6: value 1K0 -> 1K8
- R7: value 1K0 -> 3K3
